Commit message: Controllers successfully loaded and activated.

File: src/arm_description/urdf/arm_control.xacro (robot description, xacro)
@@ -2,7 +2,7 @@
 <robot xmlns:xacro="http://www.ros.org/wiki/xacro" name="robotarm">
     <xacro:property name="PI" value="3.14159"/>
-    <ros2_control type = "system" name = "GazeboSimSystem">
+    <ros2_control name="GazeboSimSystem" type="system">
         <hardware>
-            <plugin> gz_ros2_control/GazeboSimSystem</plugin>
+            <plugin>gz_ros2_control/GazeboSimSystem</plugin>
         </hardware>
         <joint name = "joint_1">
@@ -11,6 +11,5 @@
                 <param name = "max">${PI/2}</param>
             </command_interface>
-            <state_interface name = "position">
-            </state_interface>
+            <state_interface name = "position"/>
         </joint>
         <joint name = "joint_2">
@@ -19,6 +18,5 @@
                 <param name = "max">${PI/2}</param>
             </command_interface>
-            <state_interface name = "position">
-            </state_interface>
+            <state_interface name = "position"/>
         </joint>
         <joint name = "joint_3">
@@ -27,6 +25,5 @@
                 <param name = "max">${PI/2}</param>
             </command_interface>
-            <state_interface name = "position">
-            </state_interface>
+            <state_interface name = "position"/>
         </joint>
         <joint name = "joint_4">
@@ -35,6 +32,5 @@
                 <param name = "max">${PI/2}</param>
             </command_interface>
-            <state_interface name = "position">
-            </state_interface>
+            <state_interface name = "position"/>
         </joint>
         <joint name = "joint_5">
@@ -43,11 +39,10 @@
                 <param name = "max">0.0</param>
             </command_interface>
-            <state_interface name = "position">
-            </state_interface>
+            <state_interface name = "position"/>
         </joint>
-        <joint name = "joint_6">
+        <!--<joint name = "joint_6">
             <param name ="mimic">joint_5</param>
             <param name ="multiplier">-1</param>
-        </joint>
+        </joint>-->
     </ros2_control>
 </robot>

File: src/arm_description/urdf/arm_gazebo.xacro (robot description, xacro)
@@ -2,7 +2,7 @@
 <robot xmlns:xacro="http://www.ros.org/wiki/xacro" name="robotarm">
     <gazebo>
-        <plugin filename="gz_ros2_control-system" name="gz_ros2_control::GazeboSimROS2ControlPlugin">
-            <parameters>$(find arm_controller)/config/arm_controllers.yaml</parameters>
-        </plugin>
-    </gazebo>
+    <plugin filename="gz_ros2_control-system" name="gz_ros2_control::GazeboSimROS2ControlPlugin">
+      <parameters>$(find arm_controller)/config/arm_controllers.yaml</parameters>
+    </plugin>
+  </gazebo>
 </robot>

File: src/arm_description/urdf/arm_new.urdf.xacro (robot description, xacro)
@@ -1,7 +1,4 @@
 <?xml version="1.0"?>
 <robot xmlns:xacro="http://www.ros.org/wiki/xacro" name="robotarm">
-    <xacro:arg name= "is_ignition" default = "true"/>
-    <xacro:include filename="$(find arm_description)/urdf/arm_gazebo.xacro" />
-    <xacro:include filename="$(find arm_description)/urdf/arm_control.xacro" />
     <xacro:property name="PI" value="3.14159"/>
     <xacro:property name = "effort" value = "30.0"/>
@@ -187,3 +184,5 @@
         <limit lower = "0.0" upper = "${PI/2}" effort = "${effort}" velocity = "${velocity}"/>
     </joint>
+    <xacro:include filename="$(find arm_description)/urdf/arm_control.xacro" />
+    <xacro:include filename="$(find arm_description)/urdf/arm_gazebo.xacro" />
 </robot>
